Commit message: refactoring complete. display and gazebo fully functional

File: urdf/asy_robotic_arm_2026.urdf (robot description, URDF)
Before this commit: robot asy_robotic_arm_2026, 7 links, 6 joints
Links:
- added link dummy
- link End_effector: geometry collision mesh filename=package://uvic_rover/meshes/End_effector.STL; visual mesh filename=package://uvic_rover/meshes/End_effector.STL
- link Link1: geometry collision mesh filename=package://uvic_rover/meshes/Link1.STL; visual mesh filename=package://uvic_rover/meshes/Link1.STL
- link Link2: geometry collision mesh filename=package://uvic_rover/meshes/Link2.STL; visual mesh filename=package://uvic_rover/meshes/Link2.STL
- link Link3: geometry collision mesh filename=package://uvic_rover/meshes/Link3.STL; visual mesh filename=package://uvic_rover/meshes/Link3.STL
- link Link4: geometry collision mesh filename=package://uvic_rover/meshes/Link4.STL; visual mesh filename=package://uvic_rover/meshes/Link4.STL
- link Link5: geometry collision mesh filename=package://uvic_rover/meshes/Link5.STL; visual mesh filename=package://uvic_rover/meshes/Link5.STL
- link base_link: geometry collision mesh filename=package://uvic_rover/meshes/base_link.STL; visual mesh filename=package://uvic_rover/meshes/base_link.STL
Joints:
- added joint dummy_joint: type fixed, parent dummy, child base_link
- joint joint5: axis 0 0 0 -> 0 0 1

Commit message: fixed joint 4 rotation error

File: urdf/asy_robotic_arm_2026.urdf (robot description, URDF)
Before this commit: robot uvic_rover, 8 links, 7 joints
Joints:
- joint joint4: axis 0 0 1 -> 0 0 0; type continuous -> fixed

Commit message: fixed the urdf file, reused from last year

File: urdf/asy_robotic_arm_2026.urdf (robot description, URDF)
Before this commit: robot uvic_rover, 8 links, 7 joints
Links:
- removed link End_effector
- removed link Link1
- removed link Link2
- removed link Link3
- removed link Link4
- removed link Link5
- added link end_effector, mass 0.40215; collision mesh filename=package://uvicarm2024/meshes/end_effector.STL; visual mesh filename=package://uvicarm2024/meshes/end_effector.STL
- added link link1, mass 0.32157; collision mesh filename=package://uvicarm2024/meshes/link1.STL; visual mesh filename=package://uvicarm2024/meshes/link1.STL
- added link link2, mass 1.1397; collision mesh filename=package://uvicarm2024/meshes/link2.STL; visual mesh filename=package://uvicarm2024/meshes/link2.STL
- added link link3, mass 0.24583; collision mesh filename=package://uvicarm2024/meshes/link3.STL; visual mesh filename=package://uvicarm2024/meshes/link3.STL
- added link link4, mass 0.18633; collision mesh filename=package://uvicarm2024/meshes/link4.STL; visual mesh filename=package://uvicarm2024/meshes/link4.STL
- added link link5, mass 0.14869; collision mesh filename=package://uvicarm2024/meshes/link5.STL; visual mesh filename=package://uvicarm2024/meshes/link5.STL
- link base_link: geometry collision mesh filename=package://uvicarm2024/meshes/base_link.STL; visual mesh filename=package://uvicarm2024/meshes/base_link.STL
Joints:
- removed joint joint5
- removed joint joint_end_effector
- added joint end_effector_joint: type continuous, parent link5, child end_effector, origin xyz=0 0 -0.0385 rpy=3.1416 0 -1.5708, axis 0 0 1, limit effort=10 velocity=1
- added joint joint0: type continuous, parent base_link, child link1, origin xyz=0 0 0.007 rpy=1.5708 0 0, axis 0 1 0, limit effort=50 velocity=1
- joint joint1: axis 0 0 0 -> 0 0 1; child Link1 -> link2; limit (none) -> lower=0 upper=3.14 effort=50 velocity=1; origin xyz=0 0 0.0643 rpy=3.1416 0 -1.5708 -> xyz=0 0.0705 0.049 rpy=0 0 1.5708; parent base_link -> link1; type fixed -> revolute
- joint joint2: axis 0 0 1 -> 0 1 0; child Link2 -> link3; limit (none) -> effort=50 velocity=1; origin xyz=-0.00025883 0.04747 -0.0132 rpy=1.5708 1.5284 0.0054525 -> xyz=0.32 0 0 rpy=-1.5708 0 0; parent Link1 -> link2
- joint joint3: child Link3 -> link4; limit (none) -> effort=10 velocity=1; origin xyz=0.27765 0.1603 0 rpy=-3.1416 0 1.5284 -> xyz=0 0.029 -0.0575 rpy=-3.1416 0 1.5708; parent Link2 -> link3
- joint joint4: axis 0 0 0 -> 0 1 0; child Link4 -> link5; limit (none) -> effort=10 velocity=1; origin xyz=0.053502 0 -0.035471 rpy=3.1416 1.5708 3.1416 -> xyz=0 0 0.222 rpy=3.1416 0 -1.5708; parent Link3 -> link4; type fixed -> continuous

Commit message: fixed package issues

File: urdf/asy_robotic_arm_2026.urdf (robot description, URDF)
Before this commit: robot ASY, ROBOTIC ARM 2024, URDF, 8 links, 7 joints
Links:
- link base_link: geometry collision mesh filename=package://uvic_rover/meshes/base_link.STL; visual mesh filename=package://uvic_rover/meshes/base_link.STL
- link end_effector: geometry collision mesh filename=package://uvic_rover/meshes/end_effector.STL; visual mesh filename=package://uvic_rover/meshes/end_effector.STL
- link link1: geometry collision mesh filename=package://uvic_rover/meshes/link1.STL; visual mesh filename=package://uvic_rover/meshes/link1.STL
- link link2: geometry collision mesh filename=package://uvic_rover/meshes/link2.STL; visual mesh filename=package://uvic_rover/meshes/link2.STL
- link link3: geometry collision mesh filename=package://uvic_rover/meshes/link3.STL; visual mesh filename=package://uvic_rover/meshes/link3.STL
- link link4: geometry collision mesh filename=package://uvic_rover/meshes/link4.STL; visual mesh filename=package://uvic_rover/meshes/link4.STL
- link link5: geometry collision mesh filename=package://uvic_rover/meshes/link5.STL; visual mesh filename=package://uvic_rover/meshes/link5.STL
