Commit message: Add transmission tags; Change  joint names

File: urdf/drive/asy_drive_train_2026.urdf (robot description, URDF)
Before this commit: robot 2025_ROVER_ASY, 11 links, 10 joints
Joints:
- removed joint Left Bogie Wheel 1 Joint
- removed joint Left Bogie Wheel 2 Joint
- removed joint Left Front Wheel Joint
- removed joint Right Bogie Wheel 1 Joint
- removed joint Right Bogie Wheel 2 Joint
- removed joint Right Front Wheel Joint
- added joint Left_Bogie_Wheel_1_Joint: type continuous, parent Left Bogie, child Left Bogie Wheel 1, origin xyz=0.175945958234471 -0.0615759999999987 0.18423022948193 rpy=-1.57079632679488 -0.508707774402449 3.14159265358978, axis 0 0 1
- added joint Left_Bogie_Wheel_2_Joint: type continuous, parent Left Bogie, child Left Bogie Wheel 2, origin xyz=0.175945958234468 -0.0615760000000021 -0.184230229481933 rpy=1.57079632679486 -1.06208855239245 0, axis 0 0 1
- added joint Left_Front_Wheel_Joint: type continuous, parent Left Rocker, child Left Front Wheel, origin xyz=-0.460241876269187 -0.251142676859366 0.00300000000003453 rpy=0.346894155603661 -1.57079631189374 0.962086590127429, axis 1 0 0
- added joint Right_Bogie_Wheel_1_Joint: type continuous, parent Right Bogie, child Right Bogie Wheel 1, origin xyz=0.175945958234469 -0.0615760000000018 -0.184230229481932 rpy=1.57079632679488 -1.06208855239245 0, axis 0 0 1
- added joint Right_Bogie_Wheel_2_Joint: type continuous, parent Right Bogie, child Right Bogie Wheel 2, origin xyz=0.17594595823447 -0.0615759999999979 0.184230229481932 rpy=-1.57079632679488 -0.508707774402448 3.14159265358979, axis 0 0 1
- added joint Right_Front_Wheel_Joint: type continuous, parent Right Rocker, child Right Front Wheel, origin xyz=0.460241876269232 -0.251142676859283 0.00300000000000022 rpy=0.261799387799056 -1.5707963267949 0, axis 1 0 0

Commit message: Add drive train .yaml so rover loads in Gazebo, closing issue #58

File: urdf/drive/asy_drive_train_2026.urdf (robot description, URDF)
Before this commit: robot 2025_ROVER_ASY, 11 links, 10 joints
Links:
- added link dummy
- added link world
Joints:
- added joint dummy_joint: type fixed, parent dummy, child Chassis
- added joint world_fixed: type fixed, parent world, child dummy, origin xyz=0 0 0 rpy=0 0 0
